File: PCB and Schematic/sensing/EEE3088F Design Project.kicad_pcb (KiCad board)
At the start: 2 copper layers, 35 x 82 mm, 28 parts, among them J1 Conn_02x14_Odd_Even, Q1 2N3904, Q2 2N3904, Q3 2N3904

Commit message: Add files via upload
Parts:
- D1, D2, D3: footprint LED_THT:LED_D5.0mm_Horizontal_O6.35mm_Z3.0mm -> LED_THT:LED_D5.0mm_Horizontal_O6.35mm_Z9.0mm
- DP_1, DP_2, DP_3: footprint LED_THT:LED_D3.0mm_Horizontal_O6.35mm_Z2.0mm -> LED_THT:LED_D5.0mm_Horizontal_O6.35mm_Z3.0mm
- R1, R3: value 48 -> 47
- R2: value 48 -> 47; footprint Resistor_SMD:R_0201_0603Metric -> Resistor_THT:R_Axial_DIN0204_L3.6mm_D1.6mm_P1.90mm_Vertical
- RB1, RB2, RB3: value 5200 -> 5.1k
- R_DP_1, R_DP_2, R_DP_3: value 1.3M -> 1M
- TP1: value TestPoint -> Test1
- TP2: value TestPoint -> Test2
- moved TP3 25.3 mm to (51.9, 152.9)
- moved TP1 18.5 mm to (67.2, 95.0)
- moved D2 15.1 mm to (62.9, 117.6)
- moved QB2 12.4 mm to (64.0, 124.7)
- moved R_DP_1 12.0 mm to (61.3, 95.0)
- moved QB1 11.7 mm to (63.9, 87.8)
- moved QB3 10.3 mm to (64.9, 140.7)
- moved R_QB1 10.3 mm to (54.9, 92.0)
- moved DP_2 10.2 mm to (66.5, 117.6)
- moved Q2 9.61 mm to (66.0, 102.4)
- moved RB1 9.36 mm to (55.8, 87.2)
- moved R_DP_3 9.36 mm to (65.7, 132.4)
- moved RB2 8.25 mm to (60.8, 107.7)
- moved TP2 7.59 mm to (59.8, 128.6)
- moved R1 7.55 mm to (57.3, 82.6)
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Routing:
- net /PA3: track 143.8 -> 54.6 mm
- net Net-(Q3-Pad2): track 112.2 -> 51.1 mm
- net GND: track 18.2 -> 62.5 mm
- net /VO3: track 26.2 -> 51.6 mm
- net /BATT: track 192.3 -> 177.8 mm
- net /VO2: track 43.8 -> 29.5 mm
- net Net-(D2-Pad1): track 12.6 -> 22.4 mm
- net /PA5: track 41.1 -> 31.5 mm
- net Net-(Q1-Pad2): track 18.7 -> 9.43 mm
- net /PA4: track 41.6 -> 32.6 mm
- net Net-(Q2-Pad2): track 18.9 -> 11.0 mm
- net /VO1: track 33.8 -> 26.1 mm
- net /PE11: track 17.7 -> 11.4 mm
- net Net-(D1-Pad1): track 10.6 -> 16.1 mm
- net /PE15: track 48.8 -> 44.4 mm
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Other:
- board size 35 x 82 mm -> 22.4 x 80 mm
